Commit message: Working packages

File: our_arm_description/robots/OUR-II.URDF (robot description, URDF)
Before this commit: robot our_model, 19 links, 18 joints
Links:
- removed link base
- removed link link1
- removed link link10
- removed link link10_1
- removed link link11
- removed link link12
- removed link link1_1
- removed link link2
- removed link link2_1
- removed link link3
- removed link link4
- removed link link5
- removed link link6
- removed link link6_1
- removed link link7
- removed link link8
- removed link link8_1
- removed link link9
- removed link link9_1
- added link our_base, mass 0.548361856091445; collision mesh filename=package://our_arm_description/meshes/base.STL; visual mesh filename=package://our_arm_description/meshes/base.STL
- added link our_link1, mass 1.56830518389083; collision mesh filename=package://our_arm_description/meshes/link1.STL; visual mesh filename=package://our_arm_description/meshes/link1.STL
- added link our_link10, mass 0.771461023307645; collision mesh filename=package://our_arm_description/meshes/link10.STL; visual mesh filename=package://our_arm_description/meshes/link10.STL
- added link our_link10_1, mass 0.262543693353647; collision mesh filename=package://our_arm_description/meshes/link10_1.STL; visual mesh filename=package://our_arm_description/meshes/link10_1.STL
- added link our_link11, mass 0.195176525526982; collision mesh filename=package://our_arm_description/meshes/link11.STL; visual mesh filename=package://our_arm_description/meshes/link11.STL
- added link our_link12, mass 0.00060318578948924; collision mesh filename=package://our_arm_description/meshes/link12.STL; visual mesh filename=package://our_arm_description/meshes/link12.STL
- added link our_link1_1, mass 0.702288103180474; collision mesh filename=package://our_arm_description/meshes/link1_1.STL; visual mesh filename=package://our_arm_description/meshes/link1_1.STL
- added link our_link2, mass 1.56830518389083; collision mesh filename=package://our_arm_description/meshes/link2.STL; visual mesh filename=package://our_arm_description/meshes/link2.STL
- added link our_link2_1, mass 0.702288103180474; collision mesh filename=package://our_arm_description/meshes/link2_1.STL; visual mesh filename=package://our_arm_description/meshes/link2_1.STL
- added link our_link3, mass 0.355578779763243; collision mesh filename=package://our_arm_description/meshes/link3.STL; visual mesh filename=package://our_arm_description/meshes/link3.STL
- added link our_link4, mass 1.08193152317346; collision mesh filename=package://our_arm_description/meshes/link4.STL; visual mesh filename=package://our_arm_description/meshes/link4.STL
- added link our_link5, mass 0.355578779763243; collision mesh filename=package://our_arm_description/meshes/link5.STL; visual mesh filename=package://our_arm_description/meshes/link5.STL
- added link our_link6, mass 1.5683; collision mesh filename=package://our_arm_description/meshes/link6.STL; visual mesh filename=package://our_arm_description/meshes/link6.STL
- added link our_link6_1, mass 0.702288103180474; collision mesh filename=package://our_arm_description/meshes/link6_1.STL; visual mesh filename=package://our_arm_description/meshes/link6_1.STL
- added link our_link7, mass 1.78622725276023; collision mesh filename=package://our_arm_description/meshes/link7.STL; visual mesh filename=package://our_arm_description/meshes/link7.STL
- added link our_link8, mass 0.771461023307643; collision mesh filename=package://our_arm_description/meshes/link8.STL; visual mesh filename=package://our_arm_description/meshes/link8.STL
- added link our_link8_1, mass 0.262543693353647; collision mesh filename=package://our_arm_description/meshes/link8_1.STL; visual mesh filename=package://our_arm_description/meshes/link8_1.STL
- added link our_link9, mass 0.771461023307645; collision mesh filename=package://our_arm_description/meshes/link9.STL; visual mesh filename=package://our_arm_description/meshes/link9.STL
- added link our_link9_1, mass 0.262543693353647; collision mesh filename=package://our_arm_description/meshes/link9_1.STL; visual mesh filename=package://our_arm_description/meshes/link9_1.STL
Joints:
- removed joint joint03
- removed joint joint04
- removed joint joint05
- removed joint joint06
- removed joint joint1
- removed joint joint10_1
- removed joint joint12
- removed joint joint1_1
- removed joint joint2
- removed joint joint2_1
- removed joint joint3
- removed joint joint4
- removed joint joint5
- removed joint joint6
- removed joint joint6_1
- removed joint joint8
- removed joint joint8_1
- removed joint joint9_1
- added joint our_joint03: type fixed, parent our_link2, child our_link3, origin xyz=0 0.084 -0.063 rpy=3.14159265358979 0 0, axis 0 0 0
- added joint our_joint04: type fixed, parent our_link3, child our_link4, origin xyz=0 0 0.04 rpy=0 0 0, axis 0 0 0
- added joint our_joint05: type fixed, parent our_link4, child our_link5, origin xyz=0 0 0.182 rpy=0 0 0, axis 0 0 0
- added joint our_joint06: type fixed, parent our_link5, child our_link6, origin xyz=0 0 0.0400000000000001 rpy=0 0 0, axis 0 0 0
- added joint our_joint1: type revolute, parent our_base, child our_link1, origin xyz=0 0 0.024 rpy=0 0 0, axis 0 0 -1, limit lower=-1.57 upper=1.57 effort=0 velocity=0
- added joint our_joint10_1: type fixed, parent our_link10, child our_link10_1, origin xyz=0 0 0 rpy=0 0 0, axis 0 0 0
- added joint our_joint12: type fixed, parent our_link11, child our_link12, origin xyz=0 0 0 rpy=0 0 0, axis 0 0 0
- added joint our_joint1_1: type fixed, parent our_link1, child our_link1_1, origin xyz=0 0 0 rpy=0 0 0, axis 0 0 0
- added joint our_joint2: type revolute, parent our_link1, child our_link2, origin xyz=0 -0.063 0.084 rpy=3.1416 0 0, axis 0 -1 0, limit lower=-1.57 upper=1.57 effort=0 velocity=0
- added joint our_joint2_1: type fixed, parent our_link2, child our_link2_1, origin xyz=0 0 0 rpy=0 0 0, axis 0 0 0
- added joint our_joint3: type revolute, parent our_link6, child our_link7, origin xyz=0 0.084 0.063 rpy=0 0 0, axis 0 -1 0, limit lower=-1.57 upper=1.57 effort=0 velocity=0
- added joint our_joint4: type revolute, parent our_link8, child our_link9, origin xyz=0 -0.0675 0.049 rpy=3.1416 0 0, axis 0 -1 0, limit lower=-1.57 upper=1.57 effort=0 velocity=0
- added joint our_joint5: type revolute, parent our_link9, child our_link10, origin xyz=0 0.049 -0.0675 rpy=3.1416 0 0, axis 0 0 -1, limit lower=-1.57 upper=1.57 effort=0 velocity=0
- added joint our_joint6: type revolute, parent our_link10, child our_link11, origin xyz=0 -0.0675 0.049 rpy=3.1416 0 0, axis 0 -1 0, limit lower=-1.57 upper=1.57 effort=0 velocity=0
- added joint our_joint6_1: type fixed, parent our_link6, child our_link6_1, origin xyz=0 0 0 rpy=0 0 0, axis 0 0 0
- added joint our_joint8: type fixed, parent our_link7, child our_link8, origin xyz=0 0.0455000000000001 0.277999693224208 rpy=0 0 0, axis 0 0 0
- added joint our_joint8_1: type fixed, parent our_link8, child our_link8_1, origin xyz=0 0 0 rpy=0 0 0, axis 0 0 0
- added joint our_joint9_1: type fixed, parent our_link9, child our_link9_1, origin xyz=0 0 0 rpy=0 0 0, axis 0 0 0

File: summit_xl_our_description/robots/summit_xl_our.urdf.xacro (robot description, xacro)
@@ -104,5 +104,5 @@
       link="base_link" />
     <child
-      link="base" />
+      link="our_base" />
     <axis
       xyz="0 0 0" />
@@ -162,11 +162,11 @@
 		</visual>
 	</link>
-	<!--joint name="effector_joint" type="fixed">
-      <parent link="link11"/>
+	<joint name="effector_joint" type="fixed">
+      <parent link="our_link11"/>
       <child link="effector_link"/>
 	  <origin
-         xyz="0.0 0.039 0.0" rpy="0.0 0.0 0.0" />
-	</joint-->
-	<!--link name="effector_link">
+         xyz="0.0 0.039 0.0" rpy="0.0 1.58 1.58" />
+	</joint>
+	<link name="effector_link">
 		<collision>
 			<origin xyz="0.0 0.0 0.0" rpy="0 0 0"/>
@@ -181,7 +181,27 @@
 			</geometry>
 		</visual>
-	</link-->
-	<!--xacro:sensor_hokuyo_urg04lx name="hokuyo_arm" parent="effector_link">
-		<origin xyz="-0.08 -0.0138560 0.137" rpy="-0.785 0 0"/>
-	</xacro:sensor_hokuyo_urg04lx-->
+	</link>
+	<xacro:sensor_hokuyo_urg04lx name="hokuyo_arm" parent="effector_link">
+		<origin xyz="-0.0327 -0.057 0.137" rpy="${PI/2.0} 0 ${-PI/6.0}"/>
+	</xacro:sensor_hokuyo_urg04lx>
+	<joint name="arm_camera_joint" type="fixed">
+      <parent link="effector_link"/>
+      <child link="arm_camera"/>
+	  <origin
+         xyz="-0.0235 0.040703 0.12365" rpy="0.0 0.0 0.0" />
+	</joint>
+	<link name="arm_camera">
+		<collision>
+			<origin xyz="0.0 0.0 0.0" rpy="0 0 0"/>
+			<geometry>
+	     		<cylinder radius="0.025" length="0.02"/>
+			</geometry>
+		</collision>
+		<visual>
+			<origin xyz="0 0 0" rpy="0 0 0"/>
+			<geometry>
+	     		<cylinder radius="0.025" length="0.02"/>
+			</geometry>
+		</visual>
+	</link>
 </robot>
