Commit message: added tank and modified description

File: summit_xl_our_description/robots/summit_xl_our.urdf.xacro (robot description, xacro)
@@ -5,9 +5,82 @@
 	<!-- ***************** -->
 	<!-- First we import all posible elements defined in the urdf.xacro files. All these elements are defined as macro:xacros -->
+	<!-- Import summit XL base elements -->
+	<xacro:include filename="$(find summit_xl_description)/urdf/bases/summit_xl_base.urdf.xacro" />
+	<!-- Import summit XL wheels -->
+	<xacro:include filename="$(find summit_xl_description)/urdf/wheels/rubber_wheel.urdf.xacro" />
 	<!-- Import Summit XL base -->
-	<!-- xacro:include filename="$(find summit_xl_description)/robots/summit_xl_nocam.urdf.xacro" / -->
-	<xacro:include filename="$(find summit_xl_description)/robots/examples/summit_xl_our.urdf.xacro" />
+	<!-- xacro:include filename="$(find summit_xl_description)/robots/examples/summit_xl_our.urdf.xacro" / -->
+	<!-- Import all available sensors -->
+	<xacro:include filename="$(find robotnik_sensors)/urdf/all_sensors.urdf.xacro" />
+	<!-- Import specific sensor -->
+	<xacro:include filename="$(find robotnik_sensors)/urdf/gps_with_mast.urdf.xacro" />
 	<!-- Import Mico Arm -->
-	<xacro:include filename="$(find OUR-I)/robots/examples/our-i.urdf.xacro" />
+	<xacro:include filename="$(find our_arm_description)/robots/examples/our-i.urdf.xacro" />
+	<!-- ***************** -->
+	<!-- Global parameters -->
+	<!-- ***************** -->
+	<xacro:property name="PI" value="3.1415926535897931"/>
+	<!-- Wheel parameters -->
+	<xacro:property name="wheel_offset_x" value="0.229" />    <!-- x,y,z in translation from base_link to the center of the wheel -->
+	<xacro:property name="wheel_offset_y" value="0.234" />
+	<xacro:property name="wheel_offset_z" value="0.0" />
+	<!-- Flag to select the high or low quality model -->
+	<xacro:property name="hq" value="true" />
+	<!-- *************** -->
+	<!-- Robots Elements -->
+	<!-- *************** -->
+	<!-- Here we create the robot elements using the xacro:macros imported at the beggining of this file -->
+	<!-- Summit XL base -->
+	<xacro:summit_xl_base name="summit_xl" publish_bf="true" hq="${hq}" />
+	<!-- Gazebo ros control pluggins -->
+	<xacro:ros_control/>
+	<!-- Gazebo skid steering pluggins -->
+	<xacro:skid_steering broadcastOdomTF="1"/>
+	<!-- WHEELS -->
+	<xacro:rubber_wheel name="front_right" parent="base_link" reflect="false" hq="${hq}">
+		<origin xyz="${wheel_offset_x} -${wheel_offset_y} ${wheel_offset_z}" rpy="0 0 0"/>
+	</xacro:rubber_wheel>
+	<xacro:rubber_wheel name="front_left" parent="base_link" reflect="true" hq="${hq}">
+		<origin xyz="${wheel_offset_x} ${wheel_offset_y} ${wheel_offset_z}" rpy="0 0 0"/>
+	</xacro:rubber_wheel>
+	<xacro:rubber_wheel name="back_left" parent="base_link" reflect="true" hq="${hq}">
+		<origin xyz="-${wheel_offset_x} ${wheel_offset_y} ${wheel_offset_z}" rpy="0 0 0"/>
+	</xacro:rubber_wheel>
+	<xacro:rubber_wheel name="back_right" parent="base_link" reflect="false" hq="${hq}">
+		<origin xyz="-${wheel_offset_x} -${wheel_offset_y} ${wheel_offset_z}" rpy="0 0 0"/>
+	</xacro:rubber_wheel>
+	<!-- SENSORS -->
+	<!-- SENSORS -->
+	<xacro:sensor_hokuyo_utm30lx name="hokuyo" parent="base_link">
+		<origin xyz="0.0 0.0 0.33" rpy="0 0 0"/>
+	</xacro:sensor_hokuyo_utm30lx>
+<!--
+	<xacro:sensor_hokuyo_urg04lx name="hokuyo1" parent="base_link">
+		<origin xyz="-0.1 0.0 0.33" rpy="0 0 0"/>
+	</xacro:sensor_hokuyo_urg04lx>
+-->
+	<xacro:sensor_axis name="camera_front" parent="base_link">
+		<origin xyz="0.19 0 0.17" rpy="0 ${15*PI/180} 0"/>
+	</xacro:sensor_axis>
+	<xacro:sensor_axis_m5013 name="camera_rear" parent="base_link">
+		<!-- origin xyz="-0.22 0 0.275" rpy="0 0 0"/ -->
+		<origin xyz="-0.35 0 0.475" rpy="${PI/2} 0.0 -${PI/2}"/>
+	</xacro:sensor_axis_m5013>
+	<xacro:sensor_imu name="imu" parent="base_link">
+		<origin xyz="-0.18 0.0 0.170" rpy="0 0 0"/>
+	</xacro:sensor_imu>
+	<xacro:sensor_gps_with_mast name="gps" parent="base_link">
+		<origin xyz="-0.22 0.155 0.625" rpy="0 0 0"/>
+	</xacro:sensor_gps_with_mast>
+<!--
+	<xacro:sensor_kinect name="kinect" parent="base_link">
+		<origin xyz="0.325 0.0 0.16" rpy="0 0 0"/>
+	</xacro:sensor_kinect>
+-->
+<!--
+	<xacro:sensor_fotonic name="fotonic" parent="base_link">
+		<origin xyz="0.3 0.0 0.24" rpy="0 0 0"/>
+	</xacro:sensor_fotonic>
+-->
 	<!-- Gazebo ros control plugins -->
 	<!-- xacro:ros_control/ -->
@@ -34,3 +107,33 @@
       xyz="0 0 0" />
   </joint>
+   <!-- Water tank -->
+   <joint name="water_tank_fix_joint" type="fixed">
+      <parent link="base_link"/>
+      <child link="water_tank_link"/>
+	  <origin
+         xyz="-0.25 0.0 0.275"
+         rpy="0.0 0.0 0.0" />
+	</joint>
+	<link name="water_tank_link">
+		<collision>
+			<origin xyz="0 0 0" rpy="0 0 0"/>
+			<geometry>
+	     		<mesh filename="package://summit_xl_our_description/meshes/water_tank.stl"/>
+			</geometry>
+			<!-- geometry>
+				<box size="0.1 0.1 0.08"/>
+			</geometry -->
+		</collision>
+		<visual>
+			<origin xyz="0 0 0" rpy="0 0 0"/>
+			<geometry>
+	     		<mesh filename="package://summit_xl_our_description/meshes/water_tank.stl"/>
+			</geometry>
+		</visual>
+		<inertial>
+			<mass value="1e-5" />
+			<origin xyz="0 0 0" rpy="0 0 0"/>
+			<inertia ixx="1e-6" ixy="0" ixz="0" iyy="1e-6" iyz="0" izz="1e-6" />
+		</inertial>
+	</link>
 </robot>

Commit message: Fixed some problem

File: summit_xl_our_description/robots/summit_xl_our.urdf.xacro (robot description, xacro)
@@ -1,4 +1,4 @@
 <?xml version="1.0"?>
-<robot name="summit_xl_our" xmlns:xacro="http://www.ros.org/wiki/xacro">
+<robot name="summit_hl_our" xmlns:xacro="http://www.ros.org/wiki/xacro">
 	<!-- ***************** -->
 	<!-- Imported elements -->
@@ -6,5 +6,5 @@
 	<!-- First we import all posible elements defined in the urdf.xacro files. All these elements are defined as macro:xacros -->
 	<!-- Import summit XL base elements -->
-	<xacro:include filename="$(find summit_xl_description)/urdf/bases/summit_xl_base.urdf.xacro" />
+	<xacro:include filename="$(find summit_xl_description)/urdf/bases/summit_xl_hl_base.urdf.xacro" />
 	<!-- Import summit XL wheels -->
 	<xacro:include filename="$(find summit_xl_description)/urdf/wheels/rubber_wheel.urdf.xacro" />
@@ -14,7 +14,7 @@
 	<xacro:include filename="$(find robotnik_sensors)/urdf/all_sensors.urdf.xacro" />
 	<!-- Import specific sensor -->
-	<xacro:include filename="$(find robotnik_sensors)/urdf/gps_with_mast.urdf.xacro" />
-	<!-- Import Mico Arm -->
-	<xacro:include filename="$(find our_arm_description)/robots/examples/our-i.urdf.xacro" />
+	<!--xacro:include filename="$(find robotnik_sensors)/urdf/gps_with_mast.urdf.xacro" /-->
+	<!-- Import OUR Arm -->
+	<xacro:include filename="$(find our_arm_description)/robots/OUR-II.URDF" />
 	<!-- ***************** -->
 	<!-- Global parameters -->
@@ -32,5 +32,5 @@
 	<!-- Here we create the robot elements using the xacro:macros imported at the beggining of this file -->
 	<!-- Summit XL base -->
-	<xacro:summit_xl_base name="summit_xl" publish_bf="true" hq="${hq}" />
+	<xacro:summit_xl_hl_base name="summit_xl_hl	" publish_bf="true" hq="${hq}" />
 	<!-- Gazebo ros control pluggins -->
 	<xacro:ros_control/>
@@ -52,7 +52,10 @@
 	<!-- SENSORS -->
 	<!-- SENSORS -->
-	<xacro:sensor_hokuyo_utm30lx name="hokuyo" parent="base_link">
-		<origin xyz="0.0 0.0 0.33" rpy="0 0 0"/>
-	</xacro:sensor_hokuyo_utm30lx>
+	<xacro:sensor_hokuyo_urg04lx name="hokuyo_front" parent="base_link">
+		<origin xyz="0.131923 0.0 0.371673" rpy="0 0 0"/>
+	</xacro:sensor_hokuyo_urg04lx>
+	<!--xacro:sensor_hokuyo_urg04lx name="hokuyo_front" parent="base_link">
+		<origin xyz="0.131923 0.0 0.371673" rpy="0 0 0"/>
+	</xacro:sensor_hokuyo_urg04lx-->
 <!--
 	<xacro:sensor_hokuyo_urg04lx name="hokuyo1" parent="base_link">
@@ -65,12 +68,12 @@
 	<xacro:sensor_axis_m5013 name="camera_rear" parent="base_link">
 		<!-- origin xyz="-0.22 0 0.275" rpy="0 0 0"/ -->
-		<origin xyz="-0.35 0 0.475" rpy="${PI/2} 0.0 -${PI/2}"/>
+		<origin xyz="-0.315077 0 0.445633" rpy="${PI/2} 0.0 -${PI/2}"/>
 	</xacro:sensor_axis_m5013>
 	<xacro:sensor_imu name="imu" parent="base_link">
 		<origin xyz="-0.18 0.0 0.170" rpy="0 0 0"/>
 	</xacro:sensor_imu>
-	<xacro:sensor_gps_with_mast name="gps" parent="base_link">
+	<!--xacro:sensor_gps_with_mast name="gps" parent="base_link">
 		<origin xyz="-0.22 0.155 0.625" rpy="0 0 0"/>
-	</xacro:sensor_gps_with_mast>
+	</xacro:sensor_gps_with_mast-->
 <!--
 	<xacro:sensor_kinect name="kinect" parent="base_link">
@@ -95,29 +98,29 @@
 	<!-- Fix arm to robot base platform -->
 	<joint
-	  name="j_base_arm"
+	  name="our_base_arm"
       type="fixed">
     <origin
-      xyz="-0.030 0.0 0.275"
+      xyz="0.005423 0.0 0.366673"
       rpy="0.0 0.0 0.0" />
     <parent
       link="base_link" />
     <child
-      link="our_base_link" />
+      link="base" />
     <axis
       xyz="0 0 0" />
   </joint>
    <!-- Water tank -->
-   <joint name="water_tank_fix_joint" type="fixed">
+   <joint name="water_tank_base_joint" type="fixed">
       <parent link="base_link"/>
-      <child link="water_tank_link"/>
+      <child link="water_tank_base_link"/>
 	  <origin
-         xyz="-0.25 0.0 0.275"
+         xyz="0.0 0.0 0.0"
          rpy="0.0 0.0 0.0" />
 	</joint>
-	<link name="water_tank_link">
+	<link name="water_tank_base_link">
 		<collision>
 			<origin xyz="0 0 0" rpy="0 0 0"/>
 			<geometry>
-	     		<mesh filename="package://summit_xl_our_description/meshes/water_tank.stl"/>
+	     		<mesh filename="package://summit_xl_our_description/meshes/tank_arm_structure.dae"/>
 			</geometry>
 			<!-- geometry>
@@ -128,5 +131,5 @@
 			<origin xyz="0 0 0" rpy="0 0 0"/>
 			<geometry>
-	     		<mesh filename="package://summit_xl_our_description/meshes/water_tank.stl"/>
+	     		<mesh filename="package://summit_xl_our_description/meshes/tank_arm_structure.dae"/>
 			</geometry>
 		</visual>
@@ -137,3 +140,27 @@
 		</inertial>
 	</link>
+	<joint name="rp_lidar_joint" type="fixed">
+      <parent link="base_link"/>
+      <child link="rp_lidar_link"/>
+	  <origin
+         xyz="-0.348077 -0.014359 0.331673"
+         rpy="0.0 0.0 0.0" />
+	</joint>
+	<link name="rp_lidar_link">
+		<collision>
+			<origin xyz="0.0 0.0 0.0" rpy="0 0 0"/>
+			<geometry>
+	     		<box size="0.07 0.0985 0.06"/>
+			</geometry>
+			<!-- geometry>
+				<box size="0.1 0.1 0.08"/>
+			</geometry -->
+		</collision>
+		<visual>
+			<origin xyz="0 0 0" rpy="0 0 0"/>
+			<geometry>
+	     		<box size="0.07 0.0985 0.06"/>
+			</geometry>
+		</visual>
+	</link>
 </robot>

Commit message: Added moveit conf

File: summit_xl_our_description/robots/summit_xl_our.urdf.xacro (robot description, xacro)
@@ -98,9 +98,7 @@
 	<!-- Fix arm to robot base platform -->
 	<joint
-	  name="our_base_arm"
-      type="fixed">
+	  name="our_base_arm" type="fixed">
     <origin
-      xyz="0.005423 0.0 0.366673"
-      rpy="0.0 0.0 0.0" />
+      xyz="0.005423 0.0 0.366673" rpy="0.0 0.0 1.58" />
     <parent
       link="base_link" />
@@ -164,3 +162,26 @@
 		</visual>
 	</link>
+	<!--joint name="effector_joint" type="fixed">
+      <parent link="link11"/>
+      <child link="effector_link"/>
+	  <origin
+         xyz="0.0 0.039 0.0" rpy="0.0 0.0 0.0" />
+	</joint-->
+	<!--link name="effector_link">
+		<collision>
+			<origin xyz="0.0 0.0 0.0" rpy="0 0 0"/>
+			<geometry>
+	     		<mesh filename="package://summit_xl_our_description/meshes/effector-fumigator.dae"/>
+			</geometry>
+		</collision>
+		<visual>
+			<origin xyz="0 0 0" rpy="0 0 0"/>
+			<geometry>
+	     		<mesh filename="package://summit_xl_our_description/meshes/effector-fumigator.dae"/>
+			</geometry>
+		</visual>
+	</link-->
+	<!--xacro:sensor_hokuyo_urg04lx name="hokuyo_arm" parent="effector_link">
+		<origin xyz="-0.08 -0.0138560 0.137" rpy="-0.785 0 0"/>
+	</xacro:sensor_hokuyo_urg04lx-->
 </robot>

Commit message: Last working files

File: summit_xl_our_description/robots/summit_xl_our.urdf.xacro (robot description, xacro)
@@ -16,5 +16,5 @@
 	<!--xacro:include filename="$(find robotnik_sensors)/urdf/gps_with_mast.urdf.xacro" /-->
 	<!-- Import OUR Arm -->
-	<xacro:include filename="$(find our_arm_description)/robots/OUR-II.URDF" />
+	<xacro:include filename="$(find our_arm_description)/robots/our_arm.urdf" />
 	<!-- ***************** -->
 	<!-- Global parameters -->
@@ -96,16 +96,8 @@
       </plugin>
     </gazebo>
-	<!-- Fix arm to robot base platform -->
-	<joint
-	  name="our_base_arm" type="fixed">
-    <origin
-      xyz="0.005423 0.0 0.366673" rpy="0.0 0.0 1.58" />
-    <parent
-      link="base_link" />
-    <child
-      link="our_base" />
-    <axis
-      xyz="0 0 0" />
-  </joint>
+    <!-- Attach arm to robot base platform -->
+	<xacro:our_arm_i5 prefix="our_" parent="base_link">
+		<origin xyz="0.005423 0.0 0.366673" rpy="0.0 0.0 0.0	"/>
+	</xacro:our_arm_i5>
    <!-- Water tank -->
    <joint name="water_tank_base_joint" type="fixed">
@@ -122,7 +114,7 @@
 	     		<mesh filename="package://summit_xl_our_description/meshes/tank_arm_structure.dae"/>
 			</geometry>
-			<!-- geometry>
+			<geometry>
 				<box size="0.1 0.1 0.08"/>
-			</geometry -->
+			</geometry>
 		</collision>
 		<visual>
@@ -138,5 +130,5 @@
 		</inertial>
 	</link>
-	<joint name="rp_lidar_joint" type="fixed">
+	<!--joint name="rp_lidar_joint" type="fixed">
       <parent link="base_link"/>
       <child link="rp_lidar_link"/>
@@ -150,9 +142,9 @@
 			<geometry>
 	     		<box size="0.07 0.0985 0.06"/>
-			</geometry>
-			<!-- geometry>
+			</geometry-->
+			<!--geometry>
 				<box size="0.1 0.1 0.08"/>
-			</geometry -->
-		</collision>
+			</geometry-->
+		<!--/collision>
 		<visual>
 			<origin xyz="0 0 0" rpy="0 0 0"/>
@@ -161,10 +153,13 @@
 			</geometry>
 		</visual>
-	</link>
-	<joint name="effector_joint" type="fixed">
-      <parent link="our_link11"/>
+	</link-->
+    <xacro:sensor_rplidar prefix="rplidar" parent="base_link">
+         <origin xyz="-0.348077 -0.014359 0.3" rpy="0 0 ${PI/2.0}"/>
+    </xacro:sensor_rplidar>
+    <joint name="effector_joint" type="fixed">
+      <parent link="our_link7"/>
       <child link="effector_link"/>
 	  <origin
-         xyz="0.0 0.039 0.0" rpy="0.0 1.58 1.58" />
+         xyz="0.039 0.0 0.0" rpy="0.0 ${-PI/2} ${PI}" />
 	</joint>
 	<link name="effector_link">
@@ -183,5 +178,5 @@
 	</link>
 	<xacro:sensor_hokuyo_urg04lx name="hokuyo_arm" parent="effector_link">
-		<origin xyz="-0.0327 -0.057 0.137" rpy="${PI/2.0} 0 ${-PI/6.0}"/>
+		<origin xyz="-0.0327 -0.057 0.137" rpy="${PI/2.0} ${-PI/2.0} ${-PI/6.0}"/> <!--origin xyz="-0.0327 -0.057 0.137" rpy="${PI/2.0} 0 ${PI/6.0}"/-->
 	</xacro:sensor_hokuyo_urg04lx>
 	<joint name="arm_camera_joint" type="fixed">
@@ -205,3 +200,83 @@
 		</visual>
 	</link>
+	<joint name="tube_holder1_joint" type="fixed">
+      <parent link="our_link2"/>
+      <child link="tube_holder1_link"/>
+	  <origin
+         xyz="-0.078 0 0.25" rpy="0.0 0.0 0.0" />
+	</joint>
+	<link name="tube_holder1_link">
+		<collision>
+			<origin xyz="0.0 0.0 0.0" rpy="0 0 0"/>
+			<geometry>
+				<box size="0.065 0.085 0.08"/>
+			</geometry>
+		</collision>
+		<visual>
+			<origin xyz="0 0 0" rpy="0 0 0"/>
+			<geometry>
+				<box size="0.065 0.085 0.08"/>
+			</geometry>
+		</visual>
+	</link>
+	<joint name="tube_holder2_joint" type="fixed">
+      <parent link="our_link3"/>
+      <child link="tube_holder2_link"/>
+	  <origin
+         xyz="-0.07 0 0.085" rpy="0.0 0.0 0.0" />
+	</joint>
+	<link name="tube_holder2_link">
+		<collision>
+			<origin xyz="0.0 0.0 0.0" rpy="0 0 0"/>
+			<geometry>
+				<box size="0.065 0.085 0.06"/>
+			</geometry>
+		</collision>
+		<visual>
+			<origin xyz="0 0 0" rpy="0 0 0"/>
+			<geometry>
+				<box size="0.065 0.085 0.06"/>
+			</geometry>
+		</visual>
+	</link>
+	<joint name="tube_holder3_joint" type="fixed">
+      <parent link="our_link3"/>
+      <child link="tube_holder3_link"/>
+	  <origin
+         xyz="-0.07 0 0.295" rpy="0.0 0.0 0.0" />
+	</joint>
+	<link name="tube_holder3_link">
+		<collision>
+			<origin xyz="0.0 0.0 0.0" rpy="0 0 0"/>
+			<geometry>
+				<box size="0.065 0.085 0.06"/>
+			</geometry>
+		</collision>
+		<visual>
+			<origin xyz="0 0 0" rpy="0 0 0"/>
+			<geometry>
+				<box size="0.065 0.085 0.06"/>
+			</geometry>
+		</visual>
+	</link>
+	<joint name="tube_holder4_joint" type="fixed">
+      <parent link="our_link1"/>
+      <child link="tube_holder4_link"/>
+	  <origin
+         xyz="-0.050 0 0.11" rpy="0.0 0.0 0.0" />
+	</joint>
+	<link name="tube_holder4_link">
+		<collision>
+			<origin xyz="0.0 0.0 0.0" rpy="0 0 0"/>
+			<geometry>
+				<box size="0.065 0.085 0.06"/>
+			</geometry>
+		</collision>
+		<visual>
+			<origin xyz="0 0 0" rpy="0 0 0"/>
+			<geometry>
+				<box size="0.065 0.085 0.06"/>
+			</geometry>
+		</visual>
+	</link>
 </robot>

Commit message: Added gps colision

File: summit_xl_our_description/robots/summit_xl_our.urdf.xacro (robot description, xacro)
@@ -76,4 +76,7 @@
 		<origin xyz="-0.22 0.155 0.625" rpy="0 0 0"/>
 	</xacro:sensor_gps_with_mast-->
+	<xacro:sensor_gps name="gps" parent="base_link">
+		<origin xyz="-0.137 -0.187 0.85" rpy="0 0 0"/>
+	</xacro:sensor_gps>
 <!--
 	<xacro:sensor_kinect name="kinect" parent="base_link">
